File: PCB/he-sensor-breakout.kicad_sch (KiCad schematic)
At the start: 3 parts, among them J1 Conn_01x03, U1 SLSS49E

Commit message: makes sensor matrix
Parts:
- added C2: 100n, Capacitor_SMD:C_0402_1005Metric, symbol Device:C
- added J2: Conn_01x03, Connector_PinHeader_2.54mm:PinHeader_1x03_P2.54mm_Vertical, symbol Connector_Generic:Conn_01x03
- added U2: SLSS49E, Package_TO_SOT_SMD:SOT-23-3, symbol Sensor_Magnetic:SS39ET
Connections:
- net GND: now also C2.1, J2.1 (Pin_1), U2.3 (GND)
- net VCC: now also C2.2, J2.3 (Pin_3), U2.1 (VCC)
- net Vout: now also J2.2 (Pin_2), U2.2 (VOUT)
Other:
- moved on the sheet: C1, J1, U1

Commit message: adds tb
Parts:
- added U3: MCP6001-OT, Package_TO_SOT_SMD:SOT-23-5, symbol Amplifier_Operational:MCP6001-OT
Changed lines of the file:
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@@
+    )
+  )
+  (symbol (lib_id "Amplifier_Operational:MCP6001-OT") (at 175.26 108.585 0) (unit 1)
+    (in_bom yes) (on_board yes) (dnp no) (fields_autoplaced)
+    (property "Reference" "U3" (at 187.96 105.1561 0)
+      (effects (font (size 1.27 1.27)))
+    )
+    (property "Value" "MCP6001-OT" (at 187.96 107.6961 0)
+      (effects (font (size 1.27 1.27)))
+    )
+    (property "Footprint" "Package_TO_SOT_SMD:SOT-23-5" (at 172.72 113.665 0)
+      (effects (font (size 1.27 1.27)) (justify left) hide)
+    )
+    (property "Datasheet" "http://ww1.microchip.com/downloads/en/DeviceDoc/21733j.pdf" (at 175.26 103.505 0)
+      (effects (font (size 1.27 1.27)) hide)
+    )
+    (pin "2")
+    (pin "5")
+    (pin "1")
+    (pin "3")
+    (pin "4")
+    (instances
+      (project "he-sensor-breakout"
+        (path "/1c4931b8-ce31-46e7-81b2-9cf79bd80c14"
+          (reference "U3") (unit 1)
+        )
+      )
     )
   )
