File: 1u/1u.kicad_pcb (KiCad board)
At the start: 2 copper layers, 19.1 x 19 mm, 24 parts, among them J1 Conn_01x01_Pin, J10 Conn_01x01_Pin, J11 Conn_01x01_Pin, J12 Conn_01x01_Pin, J13 Conn_01x01_Pin, J14 Conn_01x01_Pin, J2 Conn_01x01_Pin, J3 Conn_01x01_Pin, J4 Conn_01x01_Pin, J5 Conn_01x01_Pin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

Commit message: cleanup
Parts:
- D1: footprint prettylib:SK6812_mini_e_flipable -> prettylib:SK6812MINI_E
