File: 1u/1u.kicad_sch (KiCad schematic)
At the start: 23 parts, among them J1 Conn_01x01_Pin, J10 Conn_01x01_Pin, J11 Conn_01x01_Pin, J12 Conn_01x01_Pin, J13 Conn_01x01_Pin, J14 Conn_01x01_Pin, J2 Conn_01x01_Pin, J3 Conn_01x01_Pin, J4 Conn_01x01_Pin, J5 Conn_01x01_Pin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

Commit message: cleanup
Parts:
- D1: footprint prettylib:SK6812_mini_e_flipable -> prettylib:SK6812MINI_E
Changed lines of the file:
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@@
     (pin "1")
     (instances
-      (project "he-sensor-breakout"
+      (project "1u"
         (path "/1c4931b8-ce31-46e7-81b2-9cf79bd80c14"
           (reference "J4") (unit 1)
@@
     (pin "2")
     (instances
-      (project "he-sensor-breakout"
+      (project "1u"
         (path "/1c4931b8-ce31-46e7-81b2-9cf79bd80c14"
           (reference "R1") (unit 1)
@@
     (pin "2")
     (instances
-      (project "he-sensor-breakout"
+      (project "1u"
         (path "/1c4931b8-ce31-46e7-81b2-9cf79bd80c14"
           (reference "C3") (unit 1)
@@
     (pin "1")
     (instances
-      (project "he-sensor-breakout"
+      (project "1u"
         (path "/1c4931b8-ce31-46e7-81b2-9cf79bd80c14"
           (reference "#PWR016") (unit 1)
@@
     (pin "1")
     (instances
-      (project "he-sensor-breakout"
+      (project "1u"
         (path "/1c4931b8-ce31-46e7-81b2-9cf79bd80c14"
           (reference "J12") (unit 1)
@@
     (pin "1")
     (instances
-      (project "he-sensor-breakout"
+      (project "1u"
         (path "/1c4931b8-ce31-46e7-81b2-9cf79bd80c14"
           (reference "#PWR07") (unit 1)
@@
     (pin "1")
     (instances
-      (project "he-sensor-breakout"
+      (project "1u"
         (path "/1c4931b8-ce31-46e7-81b2-9cf79bd80c14"
           (reference "J14") (unit 1)
@@
     (pin "1")
     (instances
-      (project "he-sensor-breakout"
+      (project "1u"
         (path "/1c4931b8-ce31-46e7-81b2-9cf79bd80c14"
           (reference "#PWR04") (unit 1)
@@
     (pin "2")
     (instances
-      (project "he-sensor-breakout"
+      (project "1u"
         (path "/1c4931b8-ce31-46e7-81b2-9cf79bd80c14"
           (reference "R2") (unit 1)
@@
     (pin "1")
     (instances
-      (project "he-sensor-breakout"
+      (project "1u"
         (path "/1c4931b8-ce31-46e7-81b2-9cf79bd80c14"
           (reference "#PWR09") (unit 1)
@@
     (pin "1")
     (instances
-      (project "he-sensor-breakout"
+      (project "1u"
         (path "/1c4931b8-ce31-46e7-81b2-9cf79bd80c14"
           (reference "J6") (unit 1)
@@
     (pin "1")
     (instances
-      (project "he-sensor-breakout"
+      (project "1u"
         (path "/1c4931b8-ce31-46e7-81b2-9cf79bd80c14"
           (reference "#PWR011") (unit 1)
@@
     (pin "1")
     (instances
-      (project "he-sensor-breakout"
+      (project "1u"
         (path "/1c4931b8-ce31-46e7-81b2-9cf79bd80c14"
           (reference "J2") (unit 1)
@@
     (pin "1")
     (instances
-      (project "he-sensor-breakout"
+      (project "1u"
         (path "/1c4931b8-ce31-46e7-81b2-9cf79bd80c14"
           (reference "#PWR014") (unit 1)
@@
     (pin "1")
     (instances
-      (project "he-sensor-breakout"
+      (project "1u"
         (path "/1c4931b8-ce31-46e7-81b2-9cf79bd80c14"
           (reference "#PWR06") (unit 1)
@@
     (pin "1")
     (instances
-      (project "he-sensor-breakout"
+      (project "1u"
         (path "/1c4931b8-ce31-46e7-81b2-9cf79bd80c14"
           (reference "#PWR02") (unit 1)
@@
     (pin "1")
     (instances
-      (project "he-sensor-breakout"
+      (project "1u"
         (path "/1c4931b8-ce31-46e7-81b2-9cf79bd80c14"
           (reference "J13") (unit 1)
@@
     (pin "1")
     (instances
-      (project "he-sensor-breakout"
+      (project "1u"
         (path "/1c4931b8-ce31-46e7-81b2-9cf79bd80c14"
           (reference "#PWR012") (unit 1)
@@
     (pin "1")
     (instances
-      (project "he-sensor-breakout"
+      (project "1u"
         (path "/1c4931b8-ce31-46e7-81b2-9cf79bd80c14"
           (reference "#PWR03") (unit 1)
@@
     (pin "1")
     (instances
-      (project "he-sensor-breakout"
+      (project "1u"
         (path "/1c4931b8-ce31-46e7-81b2-9cf79bd80c14"
           (reference "J3") (unit 1)
@@
     (pin "1")
     (instances
-      (project "he-sensor-breakout"
+      (project "1u"
         (path "/1c4931b8-ce31-46e7-81b2-9cf79bd80c14"
           (reference "#PWR05") (unit 1)
@@
     (pin "1")
     (instances
-      (project "he-sensor-breakout"
+      (project "1u"
         (path "/1c4931b8-ce31-46e7-81b2-9cf79bd80c14"
           (reference "#PWR013") (unit 1)
@@
     (pin "1")
     (instances
-      (project "he-sensor-breakout"
+      (project "1u"
         (path "/1c4931b8-ce31-46e7-81b2-9cf79bd80c14"
           (reference "J1") (unit 1)
@@
     (pin "1")
     (instances
-      (project "he-sensor-breakout"
+      (project "1u"
         (path "/1c4931b8-ce31-46e7-81b2-9cf79bd80c14"
           (reference "J8") (unit 1)
@@
     (pin "2")
     (instances
-      (project "he-sensor-breakout"
+      (project "1u"
         (path "/1c4931b8-ce31-46e7-81b2-9cf79bd80c14"
           (reference "C4") (unit 1)
@@
     (pin "1")
     (instances
-      (project "he-sensor-breakout"
+      (project "1u"
         (path "/1c4931b8-ce31-46e7-81b2-9cf79bd80c14"
           (reference "J5") (unit 1)
@@
     (pin "2")
     (instances
-      (project "he-sensor-breakout"
+      (project "1u"
         (path "/1c4931b8-ce31-46e7-81b2-9cf79bd80c14"
           (reference "R3") (unit 1)
@@
     (pin "1")
     (instances
-      (project "he-sensor-breakout"
+      (project "1u"
         (path "/1c4931b8-ce31-46e7-81b2-9cf79bd80c14"
           (reference "#PWR010") (unit 1)
@@
     (pin "1")
     (instances
-      (project "he-sensor-breakout"
+      (project "1u"
         (path "/1c4931b8-ce31-46e7-81b2-9cf79bd80c14"
           (reference "#PWR015") (unit 1)
@@
     (pin "1")
     (instances
-      (project "he-sensor-breakout"
+      (project "1u"
         (path "/1c4931b8-ce31-46e7-81b2-9cf79bd80c14"
           (reference "J7") (unit 1)
@@
       (effects (font (size 1.27 1.27)))
     )
-    (property "Footprint" "prettylib:SK6812_mini_e_flipable" (at 66.04 101.6 0)
+    (property "Footprint" "prettylib:SK6812MINI_E" (at 66.04 101.6 0)
       (effects (font (size 1.27 1.27)) (justify left top) hide)
     )
@@
     (pin "4")
     (instances
-      (project "he-sensor-breakout"
+      (project "1u"
         (path "/1c4931b8-ce31-46e7-81b2-9cf79bd80c14"
           (reference "D1") (unit 1)
@@
     (pin "3")
     (instances
-      (project "he-sensor-breakout"
+      (project "1u"
         (path "/1c4931b8-ce31-46e7-81b2-9cf79bd80c14"
           (reference "U1") (unit 1)
@@
     (pin "1")
     (instances
-      (project "he-sensor-breakout"
+      (project "1u"
         (path "/1c4931b8-ce31-46e7-81b2-9cf79bd80c14"
           (reference "#PWR01") (unit 1)
@@
     (pin "1")
     (instances
-      (project "he-sensor-breakout"
+      (project "1u"
         (path "/1c4931b8-ce31-46e7-81b2-9cf79bd80c14"
           (reference "J10") (unit 1)
@@
     (pin "1")
     (instances
-      (project "he-sensor-breakout"
+      (project "1u"
         (path "/1c4931b8-ce31-46e7-81b2-9cf79bd80c14"
           (reference "J11") (unit 1)
@@
     (pin "1")
     (instances
-      (project "he-sensor-breakout"
+      (project "1u"
         (path "/1c4931b8-ce31-46e7-81b2-9cf79bd80c14"
           (reference "#PWR08") (unit 1)
@@
     (pin "2")
     (instances
-      (project "he-sensor-breakout"
+      (project "1u"
         (path "/1c4931b8-ce31-46e7-81b2-9cf79bd80c14"
           (reference "C2") (unit 1)
@@
     (pin "2")
     (instances
-      (project "he-sensor-breakout"
+      (project "1u"
         (path "/1c4931b8-ce31-46e7-81b2-9cf79bd80c14"
           (reference "C1") (unit 1)
@@
     (pin "1")
     (instances
-      (project "he-sensor-breakout"
+      (project "1u"
         (path "/1c4931b8-ce31-46e7-81b2-9cf79bd80c14"
           (reference "J9") (unit 1)

Commit message: adds copyright notice
Other:
- title: (none) -> Hallmoeba
Changed lines of the file:
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@@
 (kicad_sch (version 20230121) (generator eeschema)
   (paper "A4")
+  (title_block
+    (title "Hallmoeba")
+    (comment 3 "Licensed under CERN-OHL-S v2 or later")
+    (comment 4 "Copyright 2023 gamaPhy")
+  )
   (junction (at 113.665 71.755) (diameter 0) (color 0 0 0 0)
   )
