File: 2u_stabilizer/2u_stabilizer.kicad_pcb (KiCad board)
At the start: 2 copper layers, 38.1 x 20.2 mm, 26 parts, among them J1 Conn_01x01_Pin, J10 Conn_01x01_Pin, J11 Conn_01x01_Pin, J12 Conn_01x01_Pin, J13 Conn_01x01_Pin, J14 Conn_01x01_Pin, J2 Conn_01x01_Pin, J3 Conn_01x01_Pin, J4 Conn_01x01_Pin, J5 Conn_01x01_Pin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

Commit message: converts to 19.05x19.05mm
Parts:
- moved C1 53.6 mm to (148.1, 136.7)
- moved C2 53.6 mm to (157.1, 135.1)
- moved C3 53.6 mm to (156.1, 130.1)
- moved C4 53.6 mm to (149.6, 131.4)
- moved ? 53.6 mm to (164.3, 140.3)
- moved ? 53.6 mm to (140.5, 140.3)
- moved D1 53.6 mm to (152.4, 137.4)
- moved J1 53.6 mm to (160.0, 139.1)
- moved J10 53.6 mm to (144.8, 126.4)
- moved J11 53.6 mm to (156.2, 141.0)
- moved J12 53.6 mm to (144.8, 141.6)
- moved J13 53.6 mm to (148.6, 141.0)
- moved J14 53.6 mm to (160.0, 141.6)
- moved J2 53.6 mm to (144.8, 139.1)
- moved J3 53.6 mm to (144.8, 128.9)
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