File: hallmoeba/hallmoeba.kicad_pcb (KiCad board)
At the start: 2 copper layers, 19.1 x 19 mm, 24 parts, among them J1 Conn_01x01_Pin, J10 Conn_01x01_Pin, J11 Conn_01x01_Pin, J12 Conn_01x01_Pin, J13 Conn_01x01_Pin, J14 Conn_01x01_Pin, J2 Conn_01x01_Pin, J3 Conn_01x01_Pin, J4 Conn_01x01_Pin, J5 Conn_01x01_Pin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

Commit message: change silkscreen
Other:
- board text added: "AGND"
- board text added: "AVDD"
- board text added: "DGND"
- board text added: "DIN"
- board text added: "DOUT"
- board text added: "DVDD"
- board text added: "Hallmoeba"
- board text added: "v1"
- board text removed: "LVDD"
- board text removed: "L_GND"
- board text removed: "L_IN"
- board text removed: "L_OUT"
- board text removed: "L_VDD"
- board text removed: "S_GND"
- board text removed: "S_VDD"
